File: Shutoff switch/switch.sch (EAGLE design)
At the start: 5 parts

Commit message: Modified circuit for new switch added name and labeling
Parts:
- removed U$1: CSAIL_PUSHBUTTON, csailPushbutton:CSAIL_PUSHBUTTON
- added S1: SWITCH-MOMENTARY-2PTH, SparkFun-Electromechanical:SWITCH-MOMENTARY-2PTH
Connections:
- net N$2: now also S1.1; no longer U$1.P$2
- net VCC: now also S1.2; no longer U$1.P$1
Changed lines of the file:
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@@
 </classes>
 <parts>
-<part name="U$1" library="csailPushbutton" deviceset="CSAIL_PUSHBUTTON" device=""/>
 <part name="C1" library="SparkFun-Capacitors" deviceset="CAP" device="PTH1" value="1uF"/>
 <part name="SUPPLY1" library="SparkFun-Aesthetics" deviceset="VCC" device=""/>
@@
 <part name="SUPPLY2" library="SparkFun-Aesthetics" deviceset="VCC" device=""/>
 <part name="GND2" library="SparkFun-Aesthetics" deviceset="GND" device=""/>
+<part name="S1" library="SparkFun-Electromechanical" deviceset="SWITCH-MOMENTARY-2" device="PTH"/>
 </parts>
 <sheets>
@@
 </plain>
 <instances>
-<instance part="U$1" gate="G$1" x="50.8" y="45.72"/>
 <instance part="C1" gate="G$1" x="66.04" y="40.64"/>
 <instance part="SUPPLY1" gate="G$1" x="86.36" y="68.58"/>
@@
 <instance part="SUPPLY2" gate="G$1" x="99.06" y="58.42"/>
 <instance part="GND2" gate="1" x="66.04" y="30.48"/>
+<instance part="S1" gate="G$1" x="60.96" y="55.88" rot="R90"/>
 </instances>
 <busses>
@@
 <net name="VCC" class="0">
 <segment>
-<pinref part="U$1" gate="G$1" pin="P$1"/>
 <pinref part="SUPPLY1" gate="G$1" pin="VCC"/>
-<wire x1="66.04" y1="60.96" x2="86.36" y2="60.96" width="0.1524" layer="91"/>
+<wire x1="60.96" y1="60.96" x2="86.36" y2="60.96" width="0.1524" layer="91"/>
 <wire x1="86.36" y1="60.96" x2="86.36" y2="68.58" width="0.1524" layer="91"/>
+<pinref part="S1" gate="G$1" pin="2"/>
 </segment>
 <segment>
@@
 <segment>
 <pinref part="R1" gate="G$1" pin="2"/>
-<pinref part="U$1" gate="G$1" pin="P$2"/>
 <wire x1="86.36" y1="48.26" x2="81.28" y2="48.26" width="0.1524" layer="91"/>
 <pinref part="R2" gate="G$1" pin="2"/>
@@
 <pinref part="C1" gate="G$1" pin="1"/>
 <wire x1="66.04" y1="45.72" x2="66.04" y2="48.26" width="0.1524" layer="91"/>
+<pinref part="S1" gate="G$1" pin="1"/>
+<wire x1="60.96" y1="50.8" x2="60.96" y2="48.26" width="0.1524" layer="91"/>
+<wire x1="60.96" y1="48.26" x2="66.04" y2="48.26" width="0.1524" layer="91"/>
+<junction x="66.04" y="48.26"/>
 </segment>
 </net>
